Commit message: docs: add RViz visualization and link Gazebo integration

File: fairino_description/urdf_dual_arms/fairino3_v6_robot.prefixed.urdf.xacro (robot description, xacro)
@@ -1,541 +1,575 @@
 <?xml version="1.0"?>
 <robot xmlns:xacro="http://www.ros.org/wiki/xacro">
-  <xacro:macro name="fairino3_v6_robot_prefixed" params="prefix joint1_angle joint2_angle joint3_angle joint4_angle joint5_angle joint6_angle">
-  <link
-    name="${prefix}base_link">
-    <inertial>
-      <origin
-        xyz="-0.00049027 -0.00045095 0.032527"
-        rpy="0 0 0" />
-      <mass
-        value="0.78393" />
-      <inertia
-        ixx="0.0013854"
-        ixy="1.1455E-05"
-        ixz="-1.0642E-05"
-        iyy="0.0013849"
-        iyz="-9.7435E-06"
-        izz="0.001977" />
-    </inertial>
-    <visual>
+  <xacro:macro name="fairino3_v6_robot_prefixed"
+    params="prefix grasp_roll:=0 grasp_pitch:=0 grasp_yaw:=0">
+    <link
+      name="${prefix}base_link">
+      <inertial>
+        <origin
+          xyz="-0.00049027 -0.00045095 0.032527"
+          rpy="0 0 0" />
+        <mass
+          value="0.78393" />
+        <inertia
+          ixx="0.0013854"
+          ixy="1.1455E-05"
+          ixz="-1.0642E-05"
+          iyy="0.0013849"
+          iyz="-9.7435E-06"
+          izz="0.001977" />
+      </inertial>
+      <visual>
+        <origin
+          xyz="0 0 0"
+          rpy="0 0 0" />
+        <geometry>
+          <mesh
+            filename="package://fairino_description/meshes/fairino3_v6/base_link.STL" />
+        </geometry>
+        <material
+          name="">
+          <color
+            rgba="0.89804 0.91765 0.92941 1" />
+        </material>
+      </visual>
+      <collision>
+        <origin
+          xyz="0 0 0"
+          rpy="0 0 0" />
+        <geometry>
+          <mesh
+            filename="package://fairino_description/meshes/fairino3_v6/base_link.STL" />
+        </geometry>
+      </collision>
+    </link>
+    <gazebo reference="${prefix}base_link">
+      <static>true</static>
+      <self_collide>true</self_collide>
+    </gazebo>
+    <link
+      name="${prefix}shoulder_link">
+      <inertial>
+        <origin
+          xyz="-3.8658E-07 -0.0024176 0.13519"
+          rpy="0 0 0" />
+        <mass
+          value="2.1225" />
+        <inertia
+          ixx="0.0033227"
+          ixy="-5.0648E-08"
+          ixz="-6.3401E-09"
+          iyy="0.0032419"
+          iyz="4.3768E-05"
+          izz="0.0023129" />
+      </inertial>
+      <visual>
+        <origin
+          xyz="0 0 0"
+          rpy="0 0 0" />
+        <geometry>
+          <mesh
+            filename="package://fairino_description/meshes/fairino3_v6/shoulder_link.STL" />
+        </geometry>
+        <material
+          name="">
+          <color
+            rgba="0.89804 0.91765 0.92941 1" />
+        </material>
+      </visual>
+      <collision>
+        <origin
+          xyz="0 0 0"
+          rpy="0 0 0" />
+        <geometry>
+          <mesh
+            filename="package://fairino_description/meshes/fairino3_v6/shoulder_link.STL" />
+        </geometry>
+      </collision>
+    </link>
+    <gazebo reference="${prefix}shoulder_link">
+      <self_collide>true</self_collide>
+    </gazebo>
+    <joint
+      name="${prefix}joint1"
+      type="revolute">
       <origin
         xyz="0 0 0"
         rpy="0 0 0" />
-      <geometry>
-        <mesh
-          filename="package://fairino_description/meshes/fairino3_v6/base_link.STL" />
-      </geometry>
-      <material
-        name="">
-        <color
-          rgba="0.89804 0.91765 0.92941 1" />
-      </material>
-    </visual>
-    <collision>
+      <parent
+        link="${prefix}base_link" />
+      <child
+        link="${prefix}shoulder_link" />
+      <axis
+        xyz="0 0 1" />
+      <limit
+        lower="-3.0543"
+        upper="3.0543"
+        effort="150"
+        velocity="3.15" />
+      <calibration
+        rising="0"
+        falling="0" />
+      <dynamics
+        damping="0"
+        friction="0" />
+      <safety_controller
+        soft_lower_limit="-3.0543"
+        soft_upper_limit="3.0543"
+        k_position="15"
+        k_velocity="10" />
+    </joint>
+    <transmission name="${prefix}joint1_trans">
+      <type>transmission_interface/SimpleTransmission</type>
+      <joint name="${prefix}joint1">
+        <hardwareInterface>hardware_interface/PositionJointInterface</hardwareInterface>
+      </joint>
+      <actuator name="${prefix}joint1_motor">
+        <hardwareInterface>hardware_interface/PositionJointInterface</hardwareInterface>
+        <mechanicalReduction>1</mechanicalReduction>
+      </actuator>
+    </transmission>
+    <link
+      name="${prefix}upperarm_link">
+      <inertial>
+        <origin
+          xyz="-0.14111 3.4656E-06 0.11053"
+          rpy="0 0 0" />
+        <mass
+          value="4.8053" />
+        <inertia
+          ixx="0.0075945"
+          ixy="3.7143E-07"
+          ixz="-7.9228E-12"
+          iyy="0.0081317"
+          iyz="-1.2918E-11"
+          izz="0.0059231" />
+      </inertial>
+      <visual>
+        <origin
+          xyz="0 0 0"
+          rpy="0 0 0" />
+        <geometry>
+          <mesh
+            filename="package://fairino_description/meshes/fairino3_v6/upperarm_link.STL" />
+        </geometry>
+        <material
+          name="">
+          <color
+            rgba="0.89804 0.91765 0.92941 1" />
+        </material>
+      </visual>
+      <collision>
+        <origin
+          xyz="0 0 0"
+          rpy="0 0 0" />
+        <geometry>
+          <mesh
+            filename="package://fairino_description/meshes/fairino3_v6/upperarm_link.STL" />
+        </geometry>
+      </collision>
+    </link>
+    <gazebo reference="${prefix}upperarm_link">
+      <self_collide>true</self_collide>
+    </gazebo>
+    <joint
+      name="${prefix}joint2"
+      type="revolute">
       <origin
-        xyz="0 0 0"
+        xyz="0 0 0.14"
+        rpy="1.5708 0 0" />
+      <parent
+        link="${prefix}shoulder_link" />
+      <child
+        link="${prefix}upperarm_link" />
+      <axis
+        xyz="0 0 1" />
+      <limit
+        lower="-4.6251"
+        upper="1.4835"
+        effort="150"
+        velocity="3.15" />
+      <calibration
+        rising="0"
+        falling="0" />
+      <dynamics
+        damping="0"
+        friction="0" />
+      <safety_controller
+        soft_lower_limit="-4.6251"
+        soft_upper_limit="1.4835"
+        k_position="15"
+        k_velocity="10" />
+    </joint>
+    <transmission name="${prefix}joint2_trans">
+      <type>transmission_interface/SimpleTransmission</type>
+      <joint name="${prefix}joint2">
+        <hardwareInterface>hardware_interface/PositionJointInterface</hardwareInterface>
+      </joint>
+      <actuator name="${prefix}joint2_motor">
+        <hardwareInterface>hardware_interface/PositionJointInterface</hardwareInterface>
+        <mechanicalReduction>1</mechanicalReduction>
+      </actuator>
+    </transmission>
+    <link
+      name="${prefix}forearm_link">
+      <inertial>
+        <origin
+          xyz="-0.18987 5.2268E-06 0.0034145"
+          rpy="0 0 0" />
+        <mass
+          value="2.2312" />
+        <inertia
+          ixx="0.0028852"
+          ixy="7.3389E-07"
+          ixz="-3.5373E-05"
+          iyy="0.0035145"
+          iyz="-2.8527E-07"
+          izz="0.0029186" />
+      </inertial>
+      <visual>
+        <origin
+          xyz="0 0 0"
+          rpy="0 0 0" />
+        <geometry>
+          <mesh
+            filename="package://fairino_description/meshes/fairino3_v6/forearm_link.STL" />
+        </geometry>
+        <material
+          name="">
+          <color
+            rgba="0.89804 0.91765 0.92941 1" />
+        </material>
+      </visual>
+      <collision>
+        <origin
+          xyz="0 0 0"
+          rpy="0 0 0" />
+        <geometry>
+          <mesh
+            filename="package://fairino_description/meshes/fairino3_v6/forearm_link.STL" />
+        </geometry>
+      </collision>
+    </link>
+    <gazebo reference="${prefix}forearm_link">
+      <self_collide>true</self_collide>
+    </gazebo>
+    <joint
+      name="${prefix}joint3"
+      type="revolute">
+      <origin
+        xyz="-0.28 0 0"
         rpy="0 0 0" />
-      <geometry>
-        <mesh
-          filename="package://fairino_description/meshes/fairino3_v6/base_link.STL" />
-      </geometry>
-    </collision>
-  </link>
-  <gazebo reference="${prefix}base_link">
-    <static>true</static>
-    <self_collide>false</self_collide>
-  </gazebo>
-  <link
-    name="${prefix}shoulder_link">
-    <inertial>
+      <parent
+        link="${prefix}upperarm_link" />
+      <child
+        link="${prefix}forearm_link" />
+      <axis
+        xyz="0 0 1" />
+      <limit
+        lower="-2.8274"
+        upper="2.8274"
+        effort="150"
+        velocity="3.15" />
+      <calibration
+        rising="0"
+        falling="0" />
+      <dynamics
+        damping="0"
+        friction="0" />
+      <safety_controller
+        soft_lower_limit="-2.8274"
+        soft_upper_limit="2.8274"
+        k_position="15"
+        k_velocity="10" />
+    </joint>
+    <transmission name="${prefix}joint3_trans">
+      <type>transmission_interface/SimpleTransmission</type>
+      <joint name="${prefix}joint3">
+        <hardwareInterface>hardware_interface/PositionJointInterface</hardwareInterface>
+      </joint>
+      <actuator name="${prefix}joint3_motor">
+        <hardwareInterface>hardware_interface/PositionJointInterface</hardwareInterface>
+        <mechanicalReduction>1</mechanicalReduction>
+      </actuator>
+    </transmission>
+    <link
+      name="${prefix}wrist1_link">
+      <inertial>
+        <origin
+          xyz="4.5665E-07 -0.0034666 0.098292"
+          rpy="0 0 0" />
+        <mass
+          value="1.5961" />
+        <inertia
+          ixx="0.0020112"
+          ixy="6.8085E-09"
+          ixz="2.4945E-08"
+          iyy="0.0014524"
+          iyz="3.2511E-05"
+          izz="0.0019076" />
+      </inertial>
+      <visual>
+        <origin
+          xyz="0 0 0"
+          rpy="0 0 0" />
+        <geometry>
+          <mesh
+            filename="package://fairino_description/meshes/fairino3_v6/wrist1_link.STL" />
+        </geometry>
+        <material
+          name="">
+          <color
+            rgba="0.89804 0.91765 0.92941 1" />
+        </material>
+      </visual>
+      <collision>
+        <origin
+          xyz="0 0 0"
+          rpy="0 0 0" />
+        <geometry>
+          <mesh
+            filename="package://fairino_description/meshes/fairino3_v6/wrist1_link.STL" />
+        </geometry>
+      </collision>
+    </link>
+    <gazebo reference="${prefix}wrist1_link">
+      <self_collide>true</self_collide>
+    </gazebo>
+    <joint
+      name="${prefix}joint4"
+      type="revolute">
       <origin
-        xyz="-3.8658E-07 -0.0024176 0.13519"
+        xyz="-0.24001 0 0"
         rpy="0 0 0" />
-      <mass
-        value="2.1225" />
-      <inertia
-        ixx="0.0033227"
-        ixy="-5.0648E-08"
-        ixz="-6.3401E-09"
-        iyy="0.0032419"
-        iyz="4.3768E-05"
-        izz="0.0023129" />
-    </inertial>
-    <visual>
+      <parent
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